File: Mixer PCB/kicad/mixer board/mixer.kicad_pcb (KiCad board)
At the start: 2 copper layers, 110.5 x 114.3 mm, 101 parts, among them IC1 LB1938FA-BH, IC2 LB1938FA-BH, IC3 LB1938FA-BH, IC4 LB1938FA-BH, IC5 LB1938FA-BH, IC6 LB1938FA-BH, IC7 LB1938FA-BH, IC8 LB1938FA-BH, IC9 PCA9615DP, J1 Conn_02x13_Odd_Even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

Commit message: Add Gerber's
Other:
- board text added: "3.3V"
- board text added: "5V"
- board text added: "GND"
- board text added: "Made By Arne Van den Broeck"
- board text added: "NRST"
- board text added: "RX"
- board text added: "SWDIO"
- board text added: "SWLK"
- board text added: "TX"
Changed lines of the file:
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@@
   (general
     (thickness 1.6)
-    (drawings 9)
+    (drawings 21)
     (tracks 2022)
     (zones 0)
@@
       (drillshape 0)
       (scaleselection 1)
-      (outputdirectory "C:/Users/arne-/Desktop/Mixergerber/"))
+      (outputdirectory "../GRBR_Board/"))
   )
   (net 0 "")
@@
     )
   )
+  (gr_text "GND\n" (at 177.8 210.566) (layer F.SilkS)
+    (effects (font (size 1 1) (thickness 0.15)))
+  )
+  (gr_text 5V (at 177.292 213.106) (layer F.SilkS)
+    (effects (font (size 1 1) (thickness 0.15)))
+  )
+  (gr_text RX (at 177.292 215.9) (layer F.SilkS)
+    (effects (font (size 1 1) (thickness 0.15)))
+  )
+  (gr_text TX (at 177.292 218.44) (layer F.SilkS)
+    (effects (font (size 1 1) (thickness 0.15)))
+  )
+  (gr_text TX (at 188.722 212.09 90) (layer F.SilkS)
+    (effects (font (size 1 1) (thickness 0.15)))
+  )
+  (gr_text "RX\n" (at 186.182 212.09 90) (layer F.SilkS)
+    (effects (font (size 1 1) (thickness 0.15)))
+  )
+  (gr_text NRST (at 196.596 221.996 90) (layer F.SilkS)
+    (effects (font (size 1 1) (thickness 0.15)))
+  )
+  (gr_text "SWDIO\n" (at 194.056 222.25 90) (layer F.SilkS)
+    (effects (font (size 1 1) (thickness 0.15)))
+  )
+  (gr_text GND (at 191.516 221.488 90) (layer F.SilkS)
+    (effects (font (size 1 1) (thickness 0.15)))
+  )
+  (gr_text "SWLK\n" (at 188.976 221.996 90) (layer F.SilkS)
+    (effects (font (size 1 1) (thickness 0.15)))
+  )
+  (gr_text "3.3V\n" (at 186.436 221.742 90) (layer F.SilkS)
+    (effects (font (size 1 1) (thickness 0.15)))
+  )
+  (gr_text "Made By Arne Van den Broeck" (at 111.76 243.078) (layer F.SilkS)
+    (effects (font (size 1.5 1.5) (thickness 0.3)))
+  )
   (dimension 110.745165 (width 0.12) (layer F.SilkS)
